Commit message: Added gripper into hercules scenario.

File: smacc2_sm_reference_library/sm_hercules_1/urdf/dual_ur.urdf.xacro (robot description, xacro)
@@ -2,7 +2,8 @@
 <robot xmlns:xacro="http://wiki.ros.org/xacro" name="$(arg name)">
    <!-- robot name parameter -->
-   <xacro:arg name="name" default="ur"/>
-   <!-- import main macro -->
+   <xacro:arg name="name" default="dual_ur"/>
+   <!-- import component macros -->
    <xacro:include filename="$(find ur_description)/urdf/ur_macro.xacro"/>
+   <xacro:include filename="$(find robotiq_85_description)/urdf/robotiq_85_gripper_macro.urdf.xacro" />
    <!-- parameters -->
    <xacro:arg name="prefix" default="" />
@@ -74,4 +75,14 @@
      <origin xyz="0 ${ box_base_size/2 } 0" rpy="${pi/2} 0 ${pi}" />          <!-- position robot in the world -->
    </xacro:ur_robot>
+   <xacro:robotiq_85_gripper
+     name="port_gripper_$(arg name)"
+     prefix="port_"
+     parent="port_tool0"
+     use_fake_hardware="$(arg use_fake_hardware)"
+     fake_sensor_commands="$(arg fake_sensor_commands)"
+     gazebo_sim="$(arg gazebo_sim)"
+     ignition_sim="$(arg ignition_sim)" >
+     <origin xyz="0 0 0" rpy="0 -${pi/2} 0"/>
+   </xacro:robotiq_85_gripper>
    <!-- arm -->
    <xacro:ur_robot
@@ -95,4 +106,14 @@
      <origin xyz="0 -${ box_base_size/2 } 0" rpy="${pi/2} 0 0" />          <!-- position robot in the world -->
    </xacro:ur_robot>
+   <xacro:robotiq_85_gripper
+     name="starboard_gripper_$(arg name)"
+     prefix="starboard_"
+     parent="starboard_tool0"
+     use_fake_hardware="$(arg use_fake_hardware)"
+     fake_sensor_commands="$(arg fake_sensor_commands)"
+     gazebo_sim="$(arg gazebo_sim)"
+     ignition_sim="$(arg ignition_sim)">
+     <origin xyz="0 0 0" rpy="0 -${pi/2} 0"/>
+   </xacro:robotiq_85_gripper>
    <xacro:if value="$(arg gazebo_sim)">
      <!-- Gazebo plugins -->

File: smacc2_sm_reference_library/sm_hercules_1/urdf/hercules.urdf.xacro (robot description, xacro)
@@ -18,4 +18,6 @@
    <!-- import UR macro -->
    <xacro:include filename="$(find ur_description)/urdf/ur_macro.xacro"/>
+   <!-- import gripper macro -->
+   <xacro:include filename="$(find robotiq_85_description)/urdf/robotiq_85_gripper_macro.urdf.xacro" />
    <!-- UR parameters -->
    <xacro:arg name="prefix" default="" />
@@ -77,4 +79,14 @@
      <origin xyz="0 ${ box_base_size/2 } 0" rpy="${pi/2} 0 ${pi}" />          <!-- position robot in the world -->
    </xacro:ur_robot>
+   <xacro:robotiq_85_gripper
+     name="$(arg prefix)port_gripper_$(arg name)"
+     prefix="$(arg prefix)port_"
+     parent="$(arg prefix)port_tool0"
+     use_fake_hardware="$(arg use_fake_hardware)"
+     fake_sensor_commands="$(arg fake_sensor_commands)"
+     gazebo_sim="$(arg gazebo_sim)"
+     ignition_sim="$(arg ignition_sim)" >
+     <origin xyz="0 0 0" rpy="0 -${pi/2} 0"/>
+   </xacro:robotiq_85_gripper>
    <!-- arm -->
    <xacro:ur_robot
@@ -98,4 +110,14 @@
      <origin xyz="0 -${ box_base_size/2 } 0" rpy="${pi/2} 0 0" />          <!-- position robot in the world -->
    </xacro:ur_robot>
+   <xacro:robotiq_85_gripper
+     name="$(arg prefix)starboard_gripper_$(arg name)"
+     prefix="$(arg prefix)starboard_"
+     parent="$(arg prefix)starboard_tool0"
+     use_fake_hardware="$(arg use_fake_hardware)"
+     fake_sensor_commands="$(arg fake_sensor_commands)"
+     gazebo_sim="$(arg gazebo_sim)"
+     ignition_sim="$(arg ignition_sim)">
+     <origin xyz="0 0 0" rpy="0 -${pi/2} 0"/>
+   </xacro:robotiq_85_gripper>
    <xacro:if value="$(arg gazebo_sim)">
      <!-- Gazebo plugins -->

Commit message: Update the simulation setup to new UR parameters.

File: smacc2_sm_reference_library/sm_hercules_1/urdf/dual_ur.urdf.xacro (robot description, xacro)
@@ -21,11 +21,13 @@
    <xacro:arg name="headless_mode" default="false" />
    <!-- initial position for fake hardware -->
-   <xacro:arg name="initial_positions_file" default="$(find ur_description)/config/initial_positions.yaml"/>
+   <xacro:arg name="initial_positions_port_file" default="$(find sm_hercules_1)/config/examples/initial_positions_port_arm.yaml"/>
+   <xacro:arg name="initial_positions_starboard_file" default="$(find sm_hercules_1)/config/examples/initial_positions_starboard_arm.yaml"/>
    <!-- Simulation parameter -->
-   <xacro:arg name="gazebo_sim" default="false" />
-   <xacro:arg name="ignition_sim" default="false" />
+   <xacro:arg name="sim_gazebo" default="false" />
+   <xacro:arg name="sim_ignition" default="false" />
    <xacro:arg name="simulation_controllers" default="$(find ur_bringup)/config/ur_controllers.yaml" />
    <!-- convert to property to use substitution in function -->
-   <xacro:property name="initial_positions_file" default="$(arg initial_positions_file)"/>
+   <xacro:property name="initial_positions_port_file" default="$(arg initial_positions_port_file)"/>
+   <xacro:property name="initial_positions_starboard_file" default="$(arg initial_positions_starboard_file)"/>
    <!-- create link fixed to the "world" -->
    <link name="world" />
@@ -70,7 +72,7 @@
      fake_sensor_commands="$(arg fake_sensor_commands)"
      headless_mode="$(arg headless_mode)"
-     initial_positions="${load_yaml(initial_positions_file)}"
-     gazebo_sim="$(arg gazebo_sim)"
-     ignition_sim="$(arg ignition_sim)" >
+     initial_positions="${load_yaml(initial_positions_port_file)}"
+     sim_gazebo="$(arg sim_gazebo)"
+     sim_ignition="$(arg sim_ignition)" >
      <origin xyz="0 ${ box_base_size/2 } 0" rpy="${pi/2} 0 ${pi}" />          <!-- position robot in the world -->
    </xacro:ur_robot>
@@ -81,6 +83,6 @@
      use_fake_hardware="$(arg use_fake_hardware)"
      fake_sensor_commands="$(arg fake_sensor_commands)"
-     gazebo_sim="$(arg gazebo_sim)"
-     ignition_sim="$(arg ignition_sim)" >
+     sim_gazebo="$(arg sim_gazebo)"
+     sim_ignition="$(arg sim_ignition)" >
      <origin xyz="0 0 0" rpy="0 -${pi/2} 0"/>
    </xacro:robotiq_85_gripper>
@@ -101,7 +103,7 @@
      fake_sensor_commands="$(arg fake_sensor_commands)"
      headless_mode="$(arg headless_mode)"
-     initial_positions="${load_yaml(initial_positions_file)}"
-     gazebo_sim="$(arg gazebo_sim)"
-     ignition_sim="$(arg ignition_sim)" >
+     initial_positions="${load_yaml(initial_positions_starboard_file)}"
+     sim_gazebo="$(arg sim_gazebo)"
+     sim_ignition="$(arg sim_ignition)" >
      <origin xyz="0 -${ box_base_size/2 } 0" rpy="${pi/2} 0 0" />          <!-- position robot in the world -->
    </xacro:ur_robot>
@@ -112,9 +114,9 @@
      use_fake_hardware="$(arg use_fake_hardware)"
      fake_sensor_commands="$(arg fake_sensor_commands)"
-     gazebo_sim="$(arg gazebo_sim)"
-     ignition_sim="$(arg ignition_sim)">
+     sim_gazebo="$(arg sim_gazebo)"
+     sim_ignition="$(arg sim_ignition)">
      <origin xyz="0 0 0" rpy="0 -${pi/2} 0"/>
    </xacro:robotiq_85_gripper>
-   <xacro:if value="$(arg gazebo_sim)">
+   <xacro:if value="$(arg sim_gazebo)">
      <!-- Gazebo plugins -->
      <gazebo reference="world">
@@ -126,5 +128,5 @@
      </gazebo>
    </xacro:if>
-   <xacro:if value="$(arg ignition_sim)">
+   <xacro:if value="$(arg sim_ignition)">
      <!-- Ignition plugins -->
      <gazebo reference="world">

File: smacc2_sm_reference_library/sm_hercules_1/urdf/hercules.urdf.xacro (robot description, xacro)
@@ -9,8 +9,9 @@
    <xacro:arg name="headless_mode" default="false" />
    <!-- initial position for simulation and fake hardware -->
-   <xacro:arg name="initial_positions_file" default="$(find ur_description)/config/initial_positions.yaml"/>
+   <xacro:arg name="initial_positions_port_file" default="$(find sm_hercules_1)/config/examples/initial_positions_port_arm.yaml"/>
+   <xacro:arg name="initial_positions_starboard_file" default="$(find sm_hercules_1)/config/examples/initial_positions_starboard_arm.yaml"/>
    <!-- Simulation parameter -->
-   <xacro:arg name="gazebo_sim" default="false" />
-   <xacro:arg name="ignition_sim" default="false" />
+   <xacro:arg name="sim_gazebo" default="false" />
+   <xacro:arg name="sim_ignition" default="false" />
    <xacro:arg name="simulation_controllers" default="$(find ur_bringup)/config/ur_controllers.yaml" />
    <!-- import Husky macro -->
@@ -31,5 +32,6 @@
    <xacro:arg name="safety_k_position" default="20"/>
    <!-- convert to property to use substitution in function -->
-   <xacro:property name="initial_positions_file" default="$(arg initial_positions_file)"/>
+   <xacro:property name="initial_positions_port_file" default="$(arg initial_positions_port_file)"/>
+   <xacro:property name="initial_positions_starboard_file" default="$(arg initial_positions_starboard_file)"/>
    <!-- Load husky description -->
    <xacro:husky prefix="$(arg prefix)" />
@@ -74,7 +76,7 @@
      fake_sensor_commands="$(arg fake_sensor_commands)"
      headless_mode="$(arg headless_mode)"
-     initial_positions="${load_yaml(initial_positions_file)}"
-     gazebo_sim="$(arg gazebo_sim)"
-     ignition_sim="$(arg ignition_sim)" >
+     initial_positions="${load_yaml(initial_positions_port_file)}"
+     sim_gazebo="$(arg sim_gazebo)"
+     sim_ignition="$(arg sim_ignition)" >
      <origin xyz="0 ${ box_base_size/2 } 0" rpy="${pi/2} 0 ${pi}" />          <!-- position robot in the world -->
    </xacro:ur_robot>
@@ -85,6 +87,6 @@
      use_fake_hardware="$(arg use_fake_hardware)"
      fake_sensor_commands="$(arg fake_sensor_commands)"
-     gazebo_sim="$(arg gazebo_sim)"
-     ignition_sim="$(arg ignition_sim)" >
+     sim_gazebo="$(arg sim_gazebo)"
+     sim_ignition="$(arg sim_ignition)" >
      <origin xyz="0 0 0" rpy="0 -${pi/2} 0"/>
    </xacro:robotiq_85_gripper>
@@ -105,7 +107,7 @@
      fake_sensor_commands="$(arg fake_sensor_commands)"
      headless_mode="$(arg headless_mode)"
-     initial_positions="${load_yaml(initial_positions_file)}"
-     gazebo_sim="$(arg gazebo_sim)"
-     ignition_sim="$(arg ignition_sim)" >
+     initial_positions="${load_yaml(initial_positions_starboard_file)}"
+     sim_gazebo="$(arg sim_gazebo)"
+     sim_ignition="$(arg sim_ignition)" >
      <origin xyz="0 -${ box_base_size/2 } 0" rpy="${pi/2} 0 0" />          <!-- position robot in the world -->
    </xacro:ur_robot>
@@ -116,9 +118,9 @@
      use_fake_hardware="$(arg use_fake_hardware)"
      fake_sensor_commands="$(arg fake_sensor_commands)"
-     gazebo_sim="$(arg gazebo_sim)"
-     ignition_sim="$(arg ignition_sim)">
+     sim_gazebo="$(arg sim_gazebo)"
+     sim_ignition="$(arg sim_ignition)">
      <origin xyz="0 0 0" rpy="0 -${pi/2} 0"/>
    </xacro:robotiq_85_gripper>
-   <xacro:if value="$(arg gazebo_sim)">
+   <xacro:if value="$(arg sim_gazebo)">
      <!-- Gazebo plugins -->
      <gazebo reference="world">
@@ -130,5 +132,5 @@
      </gazebo>
    </xacro:if>
-   <xacro:if value="$(arg ignition_sim)">
+   <xacro:if value="$(arg sim_ignition)">
      <!-- Ignition plugins -->
      <gazebo reference="world">
