Commit message: barrel search updates

File: smacc2_sm_reference_library/sm_husky_barrel_search_1/urdf/turtlebot3_waffle.urdf (robot description, URDF)
Before this commit: robot turtlebot3_waffle, 13 links, 12 joints
Links:
- removed link camera_rgb_frame
- removed link camera_rgb_optical_frame
Joints:
- removed joint camera_rgb_joint
- removed joint camera_rgb_optical_joint
