Commit message: updates in navigation

File: smacc2_sm_reference_library/sm_dancebot_ue/urdf/turtlebot3_waffle.urdf (robot description, URDF)
Before this commit: robot turtlebot3_waffle, 13 links, 12 joints
Links:
- link wheel_left_link: mass 2.8498940e-02 -> 2.8498940
- link wheel_right_link: mass 2.8498940e-02 -> 2.8498940
