Commit message: Extend sm_nav2_gazebo_test_2 with a curved-path undo phase
New mission: StNavigateWithCurve drives from the spawn area to (-2.0, 2.5)
around a pillar placed directly on the straight line, recording a genuinely
curved trajectory, and StUndoCurve retraces it exactly backwards before the
existing radial pattern runs.

Environment and configuration findings baked in from the runtime campaign:
- Arena shrunk to 7x6 m so the TB3 lidar (3.5 m) always sees at least two
  walls: AMCL stays constrained everywhere the mission drives
- Odom tracker clearing thresholds set via launch parameters: the angular
  gate is disabled and the point threshold widened, otherwise CLEAR_PATH
  consumption stalls on curved trails (recorded headings vary) and the
  replanned undo plan flaps at bends
- UndoBackwardLocalPlanner runs in free navigation mode: continuous blended
  arc steering for curved retraces (straight-line mode degenerates to
  stop-spin-creep on high-curvature sections); moderate gains
- Behavior tree replans at 0.333 Hz so carrot-reset churn cannot starve
  recovery maneuvers
- Navigation states react to state-scoped EvCbSuccess/EvCbFailure behavior
  events instead of machine-scoped EvActionSucceeded component events, which
  can survive a transition and fire spuriously in the next state
- AMCL corrects every 0.1 m / 0.1 rad for smoother small corrections

Validated end to end: curve out, 26 s curved retrace home, transit, four
radial undos, StFinalState - 5/5 undo successes, ~2.9 cm median tracking
error, zero controller/planner errors.

File: smacc2_sm_reference_library/sm_nav2_gazebo_test_2/worlds/open_arena.sdf.xacro (robot description, xacro)
@@ -79,15 +79,37 @@
         <real_time_factor>1</real_time_factor>
     </physics>
-    <!-- Rectangular arena: interior x in [-5, 5], y in [-4, 4], wall height 0.5 -->
+    <!-- Single pillar forcing a curved path on the StNavigateWithCurve leg:
+         directly between the robot spawn (-2, -0.5) and the curve goal (-2, 2.5),
+         and >2.5 m away from the radial pattern around (0.5, 0) -->
+    <model name="curve_pillar">
+      <static>1</static>
+      <link name="pillar">
+        <collision name="pillar_collision">
+          <pose>-2.0 1.0 0.25 0 0 0</pose>
+          <geometry><cylinder><radius>0.35</radius><length>0.5</length></cylinder></geometry>
+        </collision>
+        <visual name="pillar_visual">
+          <pose>-2.0 1.0 0.25 0 0 0</pose>
+          <geometry><cylinder><radius>0.35</radius><length>0.5</length></cylinder></geometry>
+          <material>
+            <ambient>0.6 0.3 0.3 1</ambient>
+            <diffuse>0.6 0.3 0.3 1</diffuse>
+          </material>
+        </visual>
+      </link>
+    </model>
+    <!-- Rectangular arena: interior x in [-4.5, 2.5], y in [-2.5, 3.5], wall height 0.5.
+         Sized so the TB3 lidar (3.5 m range) always sees at least two walls: AMCL
+         stays constrained everywhere the mission drives. -->
     <model name="arena_walls">
       <static>1</static>
       <link name="walls">
         <collision name="north_collision">
-          <pose>0 4.075 0.25 0 0 0</pose>
-          <geometry><box><size>10.3 0.15 0.5</size></box></geometry>
+          <pose>-1.0 3.575 0.25 0 0 0</pose>
+          <geometry><box><size>7.6 0.15 0.5</size></box></geometry>
         </collision>
         <visual name="north_visual">
-          <pose>0 4.075 0.25 0 0 0</pose>
-          <geometry><box><size>10.3 0.15 0.5</size></box></geometry>
+          <pose>-1.0 3.575 0.25 0 0 0</pose>
+          <geometry><box><size>7.6 0.15 0.5</size></box></geometry>
           <material>
             <ambient>0.4 0.4 0.4 1</ambient>
@@ -96,10 +118,10 @@
         </visual>
         <collision name="south_collision">
-          <pose>0 -4.075 0.25 0 0 0</pose>
-          <geometry><box><size>10.3 0.15 0.5</size></box></geometry>
+          <pose>-1.0 -2.575 0.25 0 0 0</pose>
+          <geometry><box><size>7.6 0.15 0.5</size></box></geometry>
         </collision>
         <visual name="south_visual">
-          <pose>0 -4.075 0.25 0 0 0</pose>
-          <geometry><box><size>10.3 0.15 0.5</size></box></geometry>
+          <pose>-1.0 -2.575 0.25 0 0 0</pose>
+          <geometry><box><size>7.6 0.15 0.5</size></box></geometry>
           <material>
             <ambient>0.4 0.4 0.4 1</ambient>
@@ -108,10 +130,10 @@
         </visual>
         <collision name="east_collision">
-          <pose>5.075 0 0.25 0 0 0</pose>
-          <geometry><box><size>0.15 8.0 0.5</size></box></geometry>
+          <pose>2.575 0.5 0.25 0 0 0</pose>
+          <geometry><box><size>0.15 6.0 0.5</size></box></geometry>
         </collision>
         <visual name="east_visual">
-          <pose>5.075 0 0.25 0 0 0</pose>
-          <geometry><box><size>0.15 8.0 0.5</size></box></geometry>
+          <pose>2.575 0.5 0.25 0 0 0</pose>
+          <geometry><box><size>0.15 6.0 0.5</size></box></geometry>
           <material>
             <ambient>0.4 0.4 0.4 1</ambient>
@@ -120,10 +142,10 @@
         </visual>
         <collision name="west_collision">
-          <pose>-5.075 0 0.25 0 0 0</pose>
-          <geometry><box><size>0.15 8.0 0.5</size></box></geometry>
+          <pose>-4.575 0.5 0.25 0 0 0</pose>
+          <geometry><box><size>0.15 6.0 0.5</size></box></geometry>
         </collision>
         <visual name="west_visual">
-          <pose>-5.075 0 0.25 0 0 0</pose>
-          <geometry><box><size>0.15 8.0 0.5</size></box></geometry>
+          <pose>-4.575 0.5 0.25 0 0 0</pose>
+          <geometry><box><size>0.15 6.0 0.5</size></box></geometry>
           <material>
             <ambient>0.4 0.4 0.4 1</ambient>

Commit message: Expand sm_nav2_gazebo_test_2: chained double undo and F pattern phases
The mission now exercises every undo modality in one run - ten undo
navigations total:

- Chained-undo phase: two curved legs (second pillar added to force a curve
  on the P1->P2 leg), undone in sequence through the odom tracker path
  stack. Each navigation pushes the previous trail; CbUndoPathBackwards pops
  on success, restoring the earlier leg for the next undo. The first undo of
  a chain must not clearPath on exit - only the final one clears.
- F pattern phase: SsFPattern1 ported from nova_carter sm_nav2_test_7
  (templated inner states, TDirection, force-initial-orientation idiom that
  keeps rows parallel), minus the SLAM/lidar couplings: three 1.2 m east
  rays from (0.0, -1.5), each retraced backwards, 0.4 m north pitches.

Validated end to end in gazebo: 10/10 undo successes (1 curved + 2 chained +
4 radial + 3 F rays), StFinalState reached, zero navigation errors.

File: smacc2_sm_reference_library/sm_nav2_gazebo_test_2/worlds/open_arena.sdf.xacro (robot description, xacro)
@@ -99,4 +99,23 @@
       </link>
     </model>
+    <!-- Second pillar forcing a curve on the chained leg StNavigateChain2:
+         directly between P1 (-2.0, 2.5) and P2 (1.5, 2.0) -->
+    <model name="chain_pillar">
+      <static>1</static>
+      <link name="pillar2">
+        <collision name="pillar2_collision">
+          <pose>-0.25 2.25 0.25 0 0 0</pose>
+          <geometry><cylinder><radius>0.35</radius><length>0.5</length></cylinder></geometry>
+        </collision>
+        <visual name="pillar2_visual">
+          <pose>-0.25 2.25 0.25 0 0 0</pose>
+          <geometry><cylinder><radius>0.35</radius><length>0.5</length></cylinder></geometry>
+          <material>
+            <ambient>0.3 0.3 0.6 1</ambient>
+            <diffuse>0.3 0.3 0.6 1</diffuse>
+          </material>
+        </visual>
+      </link>
+    </model>
     <!-- Rectangular arena: interior x in [-4.5, 2.5], y in [-2.5, 3.5], wall height 0.5.
          Sized so the TB3 lidar (3.5 m range) always sees at least two walls: AMCL

Commit message: Visual polish for the open arena world
Shadows, sky and a warmer sun angle; brick walls from generated running-bond
textures at real brick scale (aspect-matched per wall length); concrete
arena floor with expansion joints. Textures are generated PNGs shipped in
models/open_arena_assets and resolved via GZ_SIM_RESOURCE_PATH set by the
launch file - no Fuel downloads or network dependency. The two pillars stay
solid red and blue: they are the landmarks of the two curved undo phases.

File: smacc2_sm_reference_library/sm_nav2_gazebo_test_2/worlds/open_arena.sdf.xacro (robot description, xacro)
@@ -33,5 +33,5 @@
     </plugin>
     <light name='sun' type='directional'>
-        <cast_shadows>0</cast_shadows>
+        <cast_shadows>1</cast_shadows>
         <pose>0 0 10 0 0 0</pose>
         <diffuse>0.8 0.8 0.8 1</diffuse>
@@ -43,5 +43,5 @@
             <quadratic>0.001</quadratic>
         </attenuation>
-        <direction>-0.5 0.1 -0.9</direction>
+        <direction>-0.4 0.3 -0.85</direction>
     </light>
     <model name='ground_plane'>
@@ -65,7 +65,24 @@
                 </geometry>
                 <material>
-                    <ambient>0.8 0.8 0.8 1</ambient>
-                    <diffuse>0.8 0.8 0.8 1</diffuse>
-                    <specular>0.8 0.8 0.8 1</specular>
+                    <ambient>0.75 0.74 0.72 1</ambient>
+                    <diffuse>0.75 0.74 0.72 1</diffuse>
+                    <specular>0.2 0.2 0.2 1</specular>
+                </material>
+            </visual>
+            <visual name='arena_floor'>
+                <pose>-1.0 0.5 0.001 0 0 0</pose>
+                <geometry>
+                    <plane>
+                        <normal>0 0 1</normal>
+                        <size>7.3 6.3</size>
+                    </plane>
+                </geometry>
+                <material>
+                    <diffuse>1 1 1 1</diffuse>
+                    <specular>0.15 0.15 0.15 1</specular>
+                    <pbr><metal>
+                        <albedo_map>model://open_arena_assets/materials/textures/concrete.png</albedo_map>
+                        <roughness>0.85</roughness>
+                    </metal></pbr>
                 </material>
             </visual>
@@ -73,5 +90,8 @@
     </model>
     <scene>
-      <shadows>0</shadows>
+      <shadows>1</shadows>
+      <ambient>0.55 0.55 0.55 1</ambient>
+      <background>0.65 0.78 0.9 1</background>
+      <sky></sky>
     </scene>
     <physics name='3ms' type='ode'>
@@ -132,6 +152,10 @@
           <geometry><box><size>7.6 0.15 0.5</size></box></geometry>
           <material>
-            <ambient>0.4 0.4 0.4 1</ambient>
-            <diffuse>0.4 0.4 0.4 1</diffuse>
+            <diffuse>1 1 1 1</diffuse>
+            <specular>0.1 0.1 0.1 1</specular>
+            <pbr><metal>
+              <albedo_map>model://open_arena_assets/materials/textures/wall_long.png</albedo_map>
+              <roughness>0.9</roughness>
+            </metal></pbr>
           </material>
         </visual>
@@ -144,6 +168,10 @@
           <geometry><box><size>7.6 0.15 0.5</size></box></geometry>
           <material>
-            <ambient>0.4 0.4 0.4 1</ambient>
-            <diffuse>0.4 0.4 0.4 1</diffuse>
+            <diffuse>1 1 1 1</diffuse>
+            <specular>0.1 0.1 0.1 1</specular>
+            <pbr><metal>
+              <albedo_map>model://open_arena_assets/materials/textures/wall_long.png</albedo_map>
+              <roughness>0.9</roughness>
+            </metal></pbr>
           </material>
         </visual>
@@ -156,6 +184,10 @@
           <geometry><box><size>0.15 6.0 0.5</size></box></geometry>
           <material>
-            <ambient>0.4 0.4 0.4 1</ambient>
-            <diffuse>0.4 0.4 0.4 1</diffuse>
+            <diffuse>1 1 1 1</diffuse>
+            <specular>0.1 0.1 0.1 1</specular>
+            <pbr><metal>
+              <albedo_map>model://open_arena_assets/materials/textures/wall_side.png</albedo_map>
+              <roughness>0.9</roughness>
+            </metal></pbr>
           </material>
         </visual>
@@ -168,6 +200,10 @@
           <geometry><box><size>0.15 6.0 0.5</size></box></geometry>
           <material>
-            <ambient>0.4 0.4 0.4 1</ambient>
-            <diffuse>0.4 0.4 0.4 1</diffuse>
+            <diffuse>1 1 1 1</diffuse>
+            <specular>0.1 0.1 0.1 1</specular>
+            <pbr><metal>
+              <albedo_map>model://open_arena_assets/materials/textures/wall_side.png</albedo_map>
+              <roughness>0.9</roughness>
+            </metal></pbr>
           </material>
         </visual>
